Commit message: Humble inital setup and robot + gazebo classic  sim

File: cepheus_description/models/urdf/cepheus.xacro (robot description, xacro)
@@ -1,7 +1,6 @@
 <?xml version="1.0" ?>
 <robot name="cepheus" xmlns:xacro="http://www.ros.org/wiki/xacro">
-<xacro:include filename="$(find cepheus_description)/urdf/materials.xacro" />
-<xacro:include filename="$(find cepheus_description)/urdf/cepheus.trans" />
-<xacro:include filename="$(find cepheus_description)/urdf/cepheus.gazebo" />
+<xacro:include filename="$(find cepheus_description)/models/urdf/materials.xacro" />
+<xacro:include filename="$(find cepheus_description)/models/urdf/cepheus.gazebo" />
 <link name="base_link">
   <inertial>
@@ -13,5 +12,5 @@
     <origin xyz="0 0 0" rpy="0 0 0"/>
     <geometry>
-      <mesh filename="package://cepheus_description/meshes/cepheus.dae" scale="1 1 1"/>
+      <mesh filename="file://$(find cepheus_description)/models/meshes/cepheus.dae" scale="1 1 1"/>
     </geometry>
     <material name="silver"/>
@@ -20,5 +19,5 @@
     <origin xyz="0 0 0" rpy="0 0 0"/>
     <geometry>
-      <mesh filename="package://cepheus_description/meshes/cepheus.dae" scale="1 1 1"/>
+      <mesh filename="file://$(find cepheus_description)/models/meshes/cepheus.dae" scale="1 1 1"/>
     </geometry>
   </collision>
